Commit message: Imported upstream version '1.0.6' of 'upstream'

File: urdf/lwa4p/lwa4p.gazebo.xacro (robot description, xacro)
@@ -1,4 +1,4 @@
 <?xml version="1.0"?>
-<robot xmlns:xacro="http://www.ros.org/wiki/xacro">
+<robot xmlns:xacro="http://ros.org/wiki/xacro">
   <xacro:macro name="schunk_lwa4p_gazebo" params="name">
     <gazebo reference="${name}_0_link">

File: urdf/lwa4p/lwa4p.transmission.xacro (robot description, xacro)
@@ -1,4 +1,4 @@
 <?xml version="1.0"?>
-<robot xmlns:xacro="http://www.ros.org/wiki/xacro">
+<robot xmlns:xacro="http://ros.org/wiki/xacro">
   <xacro:macro name="schunk_lwa4p_transmission" params="name">
     <transmission name="${name}_1_trans">

File: urdf/lwa4p/lwa4p.urdf.xacro (robot description, xacro)
@@ -1,15 +1,22 @@
 <?xml version="1.0"?>
-<robot xmlns:xacro="http://www.ros.org/wiki/xacro">
+<robot xmlns:xacro="http://ros.org/wiki/xacro">
   <!-- Safety offset in rad towards the hard stop of the arm -->
-  <property name="safety_offset" value="0.02"/>
+  <xacro:property name="safety_offset" value="0.02"/>
   <!-- Some additional information used by other tools -->
   <xacro:include filename="$(find schunk_canopen_driver)/urdf/lwa4p/lwa4p.gazebo.xacro" />
   <xacro:include filename="$(find schunk_canopen_driver)/urdf/lwa4p/lwa4p.transmission.xacro" />
   <xacro:include filename="$(find schunk_canopen_driver)/urdf/materials.urdf.xacro" />
+  <xacro:macro name="default_inertial" params="mass">
+    <inertial>
+      <mass value="${mass}" />
+      <inertia ixx="0.01" ixy="0" ixz="0" iyy="0.01" iyz="0" izz="0.01" />
+      <origin xyz="0 0 0" rpy="0 0 0" />
+    </inertial>
+  </xacro:macro>
   <!-- Schunk Powerball (LWA4P) Macro -->
   <xacro:macro name="schunk_lwa4p" params="parent name *origin">
     <!-- joint between base_link and arm_0_link -->
     <joint name="${name}_0_joint" type="fixed" >
-      <insert_block name="origin" />
+      <xacro:insert_block name="origin" />
       <parent link="${parent}" />
       <child link="${name}_0_link" />
@@ -44,5 +51,5 @@
      </joint>
     <link name="${name}_1_link">
-      <xacro:default_inertial/>
+      <xacro:default_inertial mass="0.29364"/>
 <!--
       <inertial>
@@ -77,5 +84,5 @@
     </joint>
     <link name="${name}_2_link">
-      <xacro:default_inertial/>
+      <xacro:default_inertial mass="0.29364"/>
 <!--
       <inertial>
@@ -109,5 +116,5 @@
     </joint>
     <link name="${name}_3_link">
-      <xacro:default_inertial/>
+      <xacro:default_inertial mass="0.29364"/>
 <!--
       <inertial>
@@ -140,5 +147,5 @@
     </joint>
     <link name="${name}_4_link">
-      <xacro:default_inertial/>
+      <xacro:default_inertial mass="0.29364"/>
 <!--
       <inertial>
@@ -171,5 +178,5 @@
     </joint>
     <link name="${name}_5_link">
-      <xacro:default_inertial/>
+      <xacro:default_inertial mass="0.29364"/>
 <!--
       <inertial>
@@ -203,5 +210,5 @@
     </joint>
     <link name="${name}_6_link">
-      <xacro:default_inertial/>
+      <xacro:default_inertial mass="0.29364"/>
 <!--
       <inertial>
